Commit message: File Cleanup:

File: simple_mtm_v2/urdf/simple_mtm_v2.urdf (robot description, URDF)
Before this commit: robot simple_mtm_v2, 17 links, 16 joints
Links:
- link base_link: geometry collision mesh filename=package://simple_mtm_v2/meshes/visual/base_link.STL; visual mesh filename=package://simple_mtm_v2/meshes/visual/base_link.STL
- link left_G1_link: geometry collision mesh filename=package://simple_mtm_v2/meshes/visual/left_G1_link.STL; visual mesh filename=package://simple_mtm_v2/meshes/visual/left_G1_link.STL
- link left_G2_link: geometry collision mesh filename=package://simple_mtm_v2/meshes/visual/left_G2_link.STL; visual mesh filename=package://simple_mtm_v2/meshes/visual/left_G2_link.STL
- link left_G3_link: geometry collision mesh filename=package://simple_mtm_v2/meshes/visual/left_G3_link.STL; visual mesh filename=package://simple_mtm_v2/meshes/visual/left_G3_link.STL
- link left_J1_link: geometry collision mesh filename=package://simple_mtm_v2/meshes/visual/left_J1_link.STL; visual mesh filename=package://simple_mtm_v2/meshes/visual/left_J1_link.STL
- link left_J2_link: geometry collision mesh filename=package://simple_mtm_v2/meshes/visual/left_J2_link.STL; visual mesh filename=package://simple_mtm_v2/meshes/visual/left_J2_link.STL
- link left_J3_link: geometry collision mesh filename=package://simple_mtm_v2/meshes/visual/left_J3_link.STL; visual mesh filename=package://simple_mtm_v2/meshes/visual/left_J3_link.STL
- link left_lever_1_link: geometry collision mesh filename=package://simple_mtm_v2/meshes/visual/left_lever_1_link.STL; visual mesh filename=package://simple_mtm_v2/meshes/visual/left_lever_1_link.STL
- link left_lever_2_link: geometry collision mesh filename=package://simple_mtm_v2/meshes/visual/left_lever_2_link.STL; visual mesh filename=package://simple_mtm_v2/meshes/visual/left_lever_2_link.STL
- link right_G1_link: geometry collision mesh filename=package://simple_mtm_v2/meshes/visual/right_G1_link.STL; visual mesh filename=package://simple_mtm_v2/meshes/visual/right_G1_link.STL
- link right_G2_link: geometry collision mesh filename=package://simple_mtm_v2/meshes/visual/right_G2_link.STL; visual mesh filename=package://simple_mtm_v2/meshes/visual/right_G2_link.STL
- link right_G3_link: geometry collision mesh filename=package://simple_mtm_v2/meshes/visual/right_G3_link.STL; visual mesh filename=package://simple_mtm_v2/meshes/visual/right_G3_link.STL
- link right_J1_link: geometry collision mesh filename=package://simple_mtm_v2/meshes/visual/right_J1_link.STL; visual mesh filename=package://simple_mtm_v2/meshes/visual/right_J1_link.STL
- link right_J2_link: geometry collision mesh filename=package://simple_mtm_v2/meshes/visual/right_J2_link.STL; visual mesh filename=package://simple_mtm_v2/meshes/visual/right_J2_link.STL
- link right_J3_link: geometry collision mesh filename=package://simple_mtm_v2/meshes/visual/right_J3_link.STL; visual mesh filename=package://simple_mtm_v2/meshes/visual/right_J3_link.STL
- link right_lever_1_link: geometry collision mesh filename=package://simple_mtm_v2/meshes/visual/right_lever_1_link.STL; visual mesh filename=package://simple_mtm_v2/meshes/visual/right_lever_1_link.STL
- link right_lever_2_link: geometry collision mesh filename=package://simple_mtm_v2/meshes/visual/right_lever_2_link.STL; visual mesh filename=package://simple_mtm_v2/meshes/visual/right_lever_2_link.STL
