Commit message: All joints working *sunglass emoji*

File: joint_testing/urdf/simple_mtm_v10.urdf (robot description, URDF)
Before this commit: robot simple_mtm_v10, 9 links, 8 joints
Links:
- removed link right_lever_1_link
- removed link right_lever_2_link
- added link right_G0_1_link, mass 0.00204075415287946; collision mesh filename=package://mtmv16/meshes/visual/right_G0_1_link.STL; visual mesh filename=package://mtmv16/meshes/visual/right_G0_1_link.STL
- added link right_G0_2_link, mass 0.00204075409890075; collision mesh filename=package://mtmv16/meshes/visual/right_G0_2_link.STL; visual mesh filename=package://mtmv16/meshes/visual/right_G0_2_link.STL
- link right_G1_link: mass 0.00625621520567208 -> 0.00625621520567231; geometry collision mesh filename=package://mtmv16/meshes/visual/right_G1_link.STL; visual mesh filename=package://mtmv16/meshes/visual/right_G1_link.STL
- link right_G2_link: mass 0.000175394578104925 -> 0.000175394578104924; geometry collision mesh filename=package://mtmv16/meshes/visual/right_G2_link.STL; visual mesh filename=package://mtmv16/meshes/visual/right_G2_link.STL
- link right_G3_link: geometry collision mesh filename=package://mtmv16/meshes/visual/right_G3_link.STL; visual mesh filename=package://mtmv16/meshes/visual/right_G3_link.STL
Joints:
- removed joint right_lever_1_joint
- removed joint right_lever_2_joint
- added joint right_G0_1_joint: type continuous, parent right_G1_link, child right_G0_1_link, origin xyz=0 -0.0843 0 rpy=-3.1218 -7.4478E-05 -3.1341, axis 0.93442 0 -0.35618
- added joint right_G0_2_link: type continuous, parent right_G1_link, child right_G0_2_link, origin xyz=0 -0.0843 0 rpy=-3.1218 -7.4478E-05 -3.1341, axis 0.93442 0 -0.35618
- joint right_G1_joint: limit lower=0 upper=0 effort=0 velocity=0 -> (none)
- joint right_G2_joint: limit lower=0 upper=0 effort=0 velocity=0 -> (none); origin xyz=-0.0139815439024298 0.00129786118054417 0.0772341692003624 rpy=-3.14159265358979 0.364174851103282 -3.14159265358979 -> xyz=0 0.02253 0 rpy=0 -0.364174851103282 3.14159265358979
- joint right_G3_joint: axis 0 1 0 -> 0 -1 0; limit lower=0 upper=0 effort=0 velocity=0 -> (none); origin xyz=0.192500000000002 0.00969999999999821 0 rpy=0 1.5707963267949 0 -> xyz=0.232499999999994 -0.000500000000001194 0 rpy=3.14159265358979 1.5707963267949 0
